Commit message: Add Ackermann steering controller and update launch files; comment out unused components

File: mobile_robot_description/urdf/ackermann_steering.xacro (robot description, xacro)
@@ -2,5 +2,5 @@
 <robot xmlns:xacro="http://www.ros.org/wiki/xacro" name="ackermann_steering">
 <gazebo>
-      <plugin
+        <plugin
         filename="gz-sim-ackermann-steering-system"
         name="gz::sim::systems::AckermannSteering">
@@ -13,6 +13,6 @@
         <kingpin_width>1.0</kingpin_width>
         <steering_limit>0.5</steering_limit>
-        <wheel_base>1.0</wheel_base>
-        <wheel_separation>0.21</wheel_separation>
+        <wheel_base>0.38</wheel_base>
+        <wheel_separation>0.281</wheel_separation>
         <wheel_radius>0.05</wheel_radius>
         <min_velocity>-1</min_velocity>
@@ -20,4 +20,19 @@
         <min_acceleration>-3</min_acceleration>
         <max_acceleration>3</max_acceleration>
+        <topic>/cmd_vel</topic>
+        <odom_topic>/odom</odom_topic>
+        <frame_id>odom</frame_id>
+        <child_frame_id>base_link</child_frame_id>
+      </plugin>
+      <plugin
+        filename="gz-sim-joint-state-publisher-system"
+        name="gz::sim::systems::JointStatePublisher">
+        <joint_name>left_steer_joint</joint_name>
+        <joint_name>right_steer_joint</joint_name>
+        <!-- Add duplicate name for testing -->
+        <joint_name>left_front_wheel_joint</joint_name>
+        <joint_name>left_rear_wheel_joint</joint_name>
+        <joint_name>right_front_wheel_joint</joint_name>
+        <joint_name>right_rear_wheel_joint</joint_name>
       </plugin>
 </gazebo>

File: mobile_robot_description/urdf/mobile_robot.urdf.xacro (robot description, xacro)
@@ -4,6 +4,6 @@
 <xacro:include filename="$(find mobile_robot_description)/urdf/materials.xacro" />
 <xacro:include filename="$(find mobile_robot_description)/urdf/mobile_robot.xacro" />
-<xacro:include filename="$(find mobile_robot_description)/urdf/camera.xacro" />
-<xacro:include filename="$(find mobile_robot_description)/urdf/lidar.xacro" />
+<!-- <xacro:include filename="$(find mobile_robot_description)/urdf/camera.xacro" /> -->
+<!-- <xacro:include filename="$(find mobile_robot_description)/urdf/lidar.xacro" /> -->
 <!-- <xacro:include filename="$(find mobile_robot_description)/urdf/diff_drive.xacro" /> -->
 <!-- <xacro:include filename="$(find mobile_robot_description)/urdf/ackermann_steering.xacro" /> -->
@@ -16,5 +16,5 @@
     <origin xyz="0.0 0.0 0.0" rpy="0.0 0.0 0.0"/>
 </joint> -->
-<joint name="camera_joint" type="fixed">
+<!-- <joint name="camera_joint" type="fixed">
     <parent link="IntelRealsense_D435_Multibody"/>
     <child link="Camera"/>
@@ -30,4 +30,4 @@
     <child link="Lidar2_link"/>
     <origin xyz="-0.015 0.0 0.06" rpy="0.0 0.0 0.0"/>
-</joint>
+</joint> -->
 </robot>
