Commit message: Add Ackermann twist publisher and update URDF configurations for lidar and diff drive

File: mobile_robot_description/urdf/diff_drive.xacro (robot description, xacro)
@@ -16,13 +16,13 @@
             <frame_id>odom</frame_id>
             <child_frame_id>sim_world</child_frame_id>
-            <odom_topic>odom</odom_topic>
+            <!-- <odom_topic>odom</odom_topic> -->
             <odom_publisher_frequency>30</odom_publisher_frequency>
             <tf_topic>/tf</tf_topic>
         </plugin>
-        <plugin filename="gz-sim-joint-state-publisher-system" name="gz::sim::systems::JointStatePublisher">
+        <!-- <plugin filename="gz-sim-joint-state-publisher-system" name="gz::sim::systems::JointStatePublisher">
             <topic>joint_states</topic>
             <joint_name>left_rear_wheel_joint</joint_name>
             <joint_name>right_rear_wheel_joint</joint_name>
-        </plugin>
+        </plugin> -->
     </gazebo>
 </robot>

File: mobile_robot_description/urdf/lidar.xacro (robot description, xacro)
@@ -5,5 +5,5 @@
     <gazebo reference="Lidar1_link">
         <sensor name="lidar1" type="gpu_lidar">
-            <gz_frame_id>Lidar1_link</gz_frame_id>
+            <gz_frame_id>sim_world</gz_frame_id>
             <topic>lidar1_scan</topic>
             <update_rate>30</update_rate>
@@ -27,5 +27,5 @@
                     <max>12</max>
                 </range>
-                <frame_id>/Lidar1_link</frame_id>
+                <frame_id>Lidar1_link</frame_id>
             </lidar>
             <alwaysOn>true</alwaysOn>
@@ -34,8 +34,8 @@
     </gazebo>
     <!-- Lidar2 -->
-    <link name="Lidar2_link"/>
+    <!-- <link name="Lidar2_link"/>
     <gazebo reference="Lidar2_link">
         <sensor name="lidar2" type="gpu_lidar">
-            <gz_frame_id>Lidar2_link</gz_frame_id>
+            <gz_frame_id>sim_world</gz_frame_id>
             <topic>lidar2_scan</topic>
             <update_rate>30</update_rate>
@@ -59,9 +59,9 @@
                     <max>12</max>
                 </range>
-                <frame_id>/Lidar2_link</frame_id>
+                <frame_id>sim_world</frame_id>
             </lidar>
             <alwaysOn>true</alwaysOn>
             <visualize>true</visualize>
         </sensor>
-    </gazebo>
+    </gazebo> -->
 </robot>

File: mobile_robot_description/urdf/mobile_robot.urdf.xacro (robot description, xacro)
@@ -5,20 +5,20 @@
 <xacro:include filename="$(find mobile_robot_description)/urdf/mobile_robot.xacro" />
 <!-- <xacro:include filename="$(find mobile_robot_description)/urdf/camera.xacro" /> -->
-<!-- <xacro:include filename="$(find mobile_robot_description)/urdf/lidar.xacro" /> -->
-<!-- <xacro:include filename="$(find mobile_robot_description)/urdf/diff_drive.xacro" /> -->
+<xacro:include filename="$(find mobile_robot_description)/urdf/lidar.xacro" />
+<xacro:include filename="$(find mobile_robot_description)/urdf/diff_drive.xacro" />
 <!-- <xacro:include filename="$(find mobile_robot_description)/urdf/ackermann_steering.xacro" /> -->
 <xacro:include filename="$(find mobile_robot_description)/urdf/gazebo.xacro" />
 <xacro:include filename="$(find mobile_robot_description)/urdf/mobile_robot.ros2_control.xacro" />
-<!-- <link name="sim_world"/>
+<link name="sim_world"/>
 <joint name="world_joint" type="fixed">
     <parent link="sim_world"/>
     <child link="base_link"/>
     <origin xyz="0.0 0.0 0.0" rpy="0.0 0.0 0.0"/>
-</joint> -->
+</joint>
 <!-- <joint name="camera_joint" type="fixed">
     <parent link="IntelRealsense_D435_Multibody"/>
     <child link="Camera"/>
     <origin xyz="0.01 0.0 0.00" rpy="0.0 0.0 0.0"/>
-</joint>
+</joint> -->
 <joint name="lidar1_joint" type="fixed">
     <parent link="Lidar1"/>
@@ -26,5 +26,5 @@
     <origin xyz="0.015 0.0 0.06" rpy="0.0 0.0 0.0"/>
 </joint>
-<joint name="lidar2_joint" type="fixed">
+<!-- <joint name="lidar2_joint" type="fixed">
     <parent link="Lidar2"/>
     <child link="Lidar2_link"/>
