Commit message: Refactor ros2_control configuration in mobile robot URDF: rename GazeboSystem to GazeboSimSystem and simplify joint command interfaces

File: mobile_robot_description/urdf/mobile_robot.ros2_control.xacro (robot description, xacro)
@@ -1,56 +1,38 @@
 <?xml version="1.0"?>
 <robot xmlns:xacro="http://www.ros.org/wiki/xacro" name="mobile_robot">
-    <ros2_control name="GazeboSystem" type="system">
+    <ros2_control name="GazeboSimSystem" type="system">
         <hardware>
             <plugin>gz_ros2_control/GazeboSimSystem</plugin>
         </hardware>
-        <joint name="left_front_wheel_joint">
-            <command_interface name="velocity">
-                <param name="min">-10</param>
-                <param name="max">10</param>
-            </command_interface>
+        <!-- <joint name="left_front_wheel_joint">
+            <command_interface name="velocity"/>
             <state_interface name="velocity"/>
             <state_interface name="position"/>
         </joint>
         <joint name="right_front_wheel_joint">
-            <command_interface name="velocity">
-                <param name="min">-10</param>
-                <param name="max">10</param>
-            </command_interface>
+            <command_interface name="velocity"/>
             <state_interface name="velocity"/>
             <state_interface name="position"/>
-        </joint>
+        </joint> -->
         <joint name="left_rear_wheel_joint">
-            <command_interface name="velocity">
-                <param name="min">-10</param>
-                <param name="max">10</param>
-            </command_interface>
+            <command_interface name="velocity"/>
             <state_interface name="velocity"/>
             <state_interface name="position"/>
         </joint>
         <joint name="right_rear_wheel_joint">
-            <command_interface name="velocity">
-                <param name="min">-10</param>
-                <param name="max">10</param>
-            </command_interface>
+            <command_interface name="velocity"/>
             <state_interface name="velocity"/>
             <state_interface name="position"/>
         </joint>
-        <!-- <joint name="left_steer_joint">
-            <command_interface name="velocity">
-                <param name="min">-10</param>
-                <param name="max">10</param>
-            </command_interface>
+        <joint name="left_steer_joint">
+            <command_interface name="position"/>
             <state_interface name="velocity"/>
             <state_interface name="position"/>
         </joint>
         <joint name="right_steer_joint">
-            <command_interface name="velocity">
-                <param name="min">-10</param>
-                <param name="max">10</param>
-            </command_interface>
+            <command_interface name="position"/>
             <state_interface name="velocity"/>
             <state_interface name="position"/>
-        </joint> -->
+        </joint>
     </ros2_control>
     <gazebo>

Commit message: Refactor mobile_robot.ros2_control.xacro to enable state interfaces for wheel joints and add ROS remappings for odometry

File: mobile_robot_description/urdf/mobile_robot.ros2_control.xacro (robot description, xacro)
@@ -5,14 +5,14 @@
             <plugin>gz_ros2_control/GazeboSimSystem</plugin>
         </hardware>
-        <!-- <joint name="left_front_wheel_joint">
-            <command_interface name="velocity"/>
+        <joint name="left_front_wheel_joint">
+            <!-- <command_interface name="velocity"/> -->
             <state_interface name="velocity"/>
             <state_interface name="position"/>
         </joint>
         <joint name="right_front_wheel_joint">
-            <command_interface name="velocity"/>
+            <!-- <command_interface name="velocity"/> -->
             <state_interface name="velocity"/>
             <state_interface name="position"/>
-        </joint> -->
+        </joint>
         <joint name="left_rear_wheel_joint">
             <command_interface name="velocity"/>
@@ -39,5 +39,8 @@
         <plugin name="gz_ros2_control::GazeboSimROS2ControlPlugin" filename="libgz_ros2_control-system.so">
             <parameters>$(find mobile_robot_description)/config/controllers.yaml</parameters>
-            <!-- <parameters>$(find articubot_one)/config/gaz_ros2_ctl_use_sim.yaml</parameters> -->
+            <ros>
+                <remapping>ackermann_steering_cont/odometry:=odom</remapping>
+                <remapping>ackermann_steering_cont/tf_odometry:=tf</remapping>
+            </ros>
         </plugin>
     </gazebo>
