Commit message: Update mobile robot URDF: adjust base link origin, add Gazebo properties, and enhance joint dynamics

File: mobile_robot_description/urdf/mobile_robot.xacro (robot description, xacro)
@@ -3,5 +3,6 @@
 <link name="base_link">
   <inertial>
-    <origin xyz="4.165113628650796e-06 0.02588707927115077 -0.004097141774192208" rpy="0 0 0"/>
+    <!-- <origin xyz="0.0 0.02588707927115077 -0.004097141774192208" rpy="0 0 0"/> -->
+    <origin xyz="0.0 0.02588707927115077 0.01097141774192208" rpy="0 0 0"/>
     <mass value="2.1479557811007264"/>
     <inertia ixx="0.017182" iyy="0.071938" izz="0.086976" ixy="0.0" iyz="0.0" ixz="1e-06"/>
@@ -301,4 +302,6 @@
   </collision>
 </link>
+<gazebo reference_link = "tyre">
+</gazebo>
 <link name="tyre3">
   <inertial>
@@ -390,4 +393,6 @@
   <child link="left_front_wheel"/>
   <axis xyz="0.0 1.0 0.0"/>
+  <limit effort="200.0" velocity="20.0"/>
+  <dynamics friction="0.0001"/>
 </joint>
 <joint name="right_front_wheel_joint" type="continuous">
@@ -396,4 +401,6 @@
   <child link="right_front_wheel"/>
   <axis xyz="0.0 1.0 0.0"/>
+  <limit effort="200.0" velocity="20.0"/>
+  <dynamics friction="1.0"/>
 </joint>
 <joint name="left_rear_wheel_joint" type="continuous">
@@ -402,4 +409,6 @@
   <child link="left_rear_wheel"/>
   <axis xyz="0.0 1.0 0.0"/>
+  <limit effort="200.0" velocity="20.0"/>
+  <dynamics damping="1.0" friction="1.0"/>
 </joint>
 <joint name="right_rear_wheel_joint" type="continuous">
@@ -408,4 +417,6 @@
   <child link="right_rear_wheel"/>
   <axis xyz="0.0 1.0 0.0"/>
+  <limit effort="200.0" velocity="20.0"/>
+  <dynamics damping="1.0" friction="1.0"/>
 </joint>
 <joint name="Rigid 23" type="fixed">

Commit message: Rename 'base_link' to 'chassis' in mobile robot URDF and update associated mesh and joint references

File: mobile_robot_description/urdf/mobile_robot.xacro (robot description, xacro)
@@ -1,5 +1,5 @@
 <?xml version="1.0" ?>
 <robot name="mobile_robot" xmlns:xacro="http://www.ros.org/wiki/xacro">
-<link name="base_link">
+<link name="chassis">
   <inertial>
     <!-- <origin xyz="0.0 0.02588707927115077 -0.004097141774192208" rpy="0 0 0"/> -->
@@ -11,5 +11,5 @@
     <origin xyz="0 0 0" rpy="0 0 0"/>
     <geometry>
-      <mesh filename="package://mobile_robot_description/meshes/base_link.stl" scale="0.001 0.001 0.001"/>
+      <mesh filename="package://mobile_robot_description/meshes/chassis.stl" scale="0.001 0.001 0.001"/>
     </geometry>
     <material name="paint_metallic_silver"/>
@@ -18,5 +18,5 @@
     <origin xyz="0 0 0" rpy="0 0 0"/>
     <geometry>
-      <mesh filename="package://mobile_robot_description/meshes/base_link.stl" scale="0.001 0.001 0.001"/>
+      <mesh filename="package://mobile_robot_description/meshes/chassis.stl" scale="0.001 0.001 0.001"/>
     </geometry>
   </collision>
@@ -346,10 +346,10 @@
 <joint name="Rigid 1" type="fixed">
   <origin xyz="0.30383 -0.009113 -0.017217" rpy="0 0 0"/>
-  <parent link="base_link"/>
+  <parent link="chassis"/>
   <child link="LidarHolder1"/>
 </joint>
 <joint name="Rigid 2" type="fixed">
   <origin xyz="-0.29617 0.060887 -0.017217" rpy="0 0 0"/>
-  <parent link="base_link"/>
+  <parent link="chassis"/>
   <child link="LidarHolder2"/>
 </joint>
@@ -366,5 +366,5 @@
 <joint name="Rigid 5" type="fixed">
   <origin xyz="0.30183 0.025887 0.022283" rpy="0 0 0"/>
-  <parent link="base_link"/>
+  <parent link="chassis"/>
   <child link="CameraHolder"/>
 </joint>
@@ -376,5 +376,5 @@
 <joint name="left_steer_joint" type="revolute">
   <origin xyz="0.19383 0.140887 -0.009717" rpy="0 0 0"/>
-  <parent link="base_link"/>
+  <parent link="chassis"/>
   <child link="Wheelbracket_1"/>
   <axis xyz="0.0 0.0 1.0"/>
@@ -383,5 +383,5 @@
 <joint name="right_steer_joint" type="revolute">
   <origin xyz="0.19383 -0.089113 -0.009717" rpy="0 0 0"/>
-  <parent link="base_link"/>
+  <parent link="chassis"/>
   <child link="Wheelbracket_2"/>
   <axis xyz="0.0 0.0 1.0"/>
@@ -406,5 +406,5 @@
 <joint name="left_rear_wheel_joint" type="continuous">
   <origin xyz="-0.18617 0.140887 -0.009717" rpy="0 0 0"/>
-  <parent link="base_link"/>
+  <parent link="chassis"/>
   <child link="left_rear_wheel"/>
   <axis xyz="0.0 1.0 0.0"/>
@@ -414,5 +414,5 @@
 <joint name="right_rear_wheel_joint" type="continuous">
   <origin xyz="-0.18617 -0.089113 -0.009717" rpy="0 0 0"/>
-  <parent link="base_link"/>
+  <parent link="chassis"/>
   <child link="right_rear_wheel"/>
   <axis xyz="0.0 1.0 0.0"/>

Commit message: Update left front wheel joint origin and adjust friction dynamics for improved performance

File: mobile_robot_description/urdf/mobile_robot.xacro (robot description, xacro)
@@ -389,5 +389,5 @@
 </joint>
 <joint name="left_front_wheel_joint" type="continuous">
-  <origin xyz="0.0 0.001 0.0" rpy="0 0 0"/>
+  <origin xyz="0.0 0.0 0.0" rpy="0 0 0"/>
   <parent link="Wheelbracket_1"/>
   <child link="left_front_wheel"/>
@@ -402,5 +402,5 @@
   <axis xyz="0.0 1.0 0.0"/>
   <limit effort="200.0" velocity="20.0"/>
-  <dynamics friction="1.0"/>
+  <dynamics friction="0.0001"/>
 </joint>
 <joint name="left_rear_wheel_joint" type="continuous">
