Commit message: Add additional sensor configurations and adjust joint origins in mobile robot URDF

File: mobile_robot_description/urdf/mobile_robot.urdf.xacro (robot description, xacro)
@@ -1,22 +1,26 @@
 <?xml version="1.0"?>
 <robot xmlns:xacro="http://www.ros.org/wiki/xacro" name="mobile_robot">
+<xacro:property name="PI" value="3.141592654"/>
 <xacro:include filename="$(find mobile_robot_description)/urdf/materials.xacro" />
 <xacro:include filename="$(find mobile_robot_description)/urdf/mobile_robot.xacro" />
 <xacro:include filename="$(find mobile_robot_description)/urdf/camera.xacro" />
 <xacro:include filename="$(find mobile_robot_description)/urdf/lidar.xacro" />
+<xacro:include filename="$(find mobile_robot_description)/urdf/diff_drive.xacro" />
+<xacro:include filename="$(find mobile_robot_description)/urdf/ackermann_steering.xacro" />
+<xacro:include filename="$(find mobile_robot_description)/urdf/mobile_robot.ros2_control.xacro" />
 <joint name="camera_joint" type="fixed">
     <parent link="IntelRealsense_D435_Multibody"/>
     <child link="Camera"/>
-    <origin xyz="0.0 0.0 0.0" rpy="0.0 0.0 0.0"/>
+    <origin xyz="0.01 0.0 0.00" rpy="0.0 0.0 0.0"/>
 </joint>
 <joint name="lidar1_joint" type="fixed">
     <parent link="Lidar1"/>
     <child link="Lidar1_link"/>
-    <origin xyz="0.0 0.0 0.0" rpy="0.0 0.0 0.0"/>
+    <origin xyz="0.015 0.0 0.06" rpy="0.0 0.0 0.0"/>
 </joint>
 <joint name="lidar2_joint" type="fixed">
     <parent link="Lidar2"/>
     <child link="Lidar2_link"/>
-    <origin xyz="0.0 0.0 0.0" rpy="0.0 0.0 0.0"/>
+    <origin xyz="-0.015 0.0 0.06" rpy="0.0 0.0 0.0"/>
 </joint>
 </robot>

Commit message: Refactor mobile robot URDF: comment out differential drive and Ackermann steering includes, add Gazebo integration

File: mobile_robot_description/urdf/mobile_robot.urdf.xacro (robot description, xacro)
@@ -6,7 +6,14 @@
 <xacro:include filename="$(find mobile_robot_description)/urdf/camera.xacro" />
 <xacro:include filename="$(find mobile_robot_description)/urdf/lidar.xacro" />
-<xacro:include filename="$(find mobile_robot_description)/urdf/diff_drive.xacro" />
-<xacro:include filename="$(find mobile_robot_description)/urdf/ackermann_steering.xacro" />
+<!-- <xacro:include filename="$(find mobile_robot_description)/urdf/diff_drive.xacro" /> -->
+<!-- <xacro:include filename="$(find mobile_robot_description)/urdf/ackermann_steering.xacro" /> -->
+<xacro:include filename="$(find mobile_robot_description)/urdf/gazebo.xacro" />
 <xacro:include filename="$(find mobile_robot_description)/urdf/mobile_robot.ros2_control.xacro" />
+<!-- <link name="sim_world"/>
+<joint name="world_joint" type="fixed">
+    <parent link="sim_world"/>
+    <child link="base_link"/>
+    <origin xyz="0.0 0.0 0.0" rpy="0.0 0.0 0.0"/>
+</joint> -->
 <joint name="camera_joint" type="fixed">
     <parent link="IntelRealsense_D435_Multibody"/>

Commit message: Update mobile robot URDF to change link name to 'base_link' and add base footprint and chassis joints

File: mobile_robot_description/urdf/mobile_robot.urdf.xacro (robot description, xacro)
@@ -10,8 +10,14 @@
 <xacro:include filename="$(find mobile_robot_description)/urdf/gazebo.xacro" />
 <xacro:include filename="$(find mobile_robot_description)/urdf/mobile_robot.ros2_control.xacro" />
-<link name="sim_world"/>
-<joint name="world_joint" type="fixed">
-    <parent link="sim_world"/>
-    <child link="base_link"/>
+<link name="base_link"/>
+<joint name="base_footprint_joint" type="fixed">
+    <parent link="base_link"/>
+    <child link="base_footprint"/>
+    <origin xyz="0.0 0.0 0.0" rpy="0.0 0.0 0.0"/>
+</joint>
+<link name="base_footprint"/>
+<joint name="chassis_joint" type="fixed">
+    <parent link="base_link"/>
+    <child link="chassis"/>
     <origin xyz="0.0 0.0 0.0" rpy="0.0 0.0 0.0"/>
 </joint>

Commit message: Update lidar joint configuration in mobile_robot.urdf.xacro for improved alignment and clarity

File: mobile_robot_description/urdf/mobile_robot.urdf.xacro (robot description, xacro)
@@ -6,5 +6,5 @@
 <!-- <xacro:include filename="$(find mobile_robot_description)/urdf/camera.xacro" /> -->
 <xacro:include filename="$(find mobile_robot_description)/urdf/lidar.xacro" />
-<xacro:include filename="$(find mobile_robot_description)/urdf/diff_drive.xacro" />
+<!-- <xacro:include filename="$(find mobile_robot_description)/urdf/diff_drive.xacro" /> -->
 <!-- <xacro:include filename="$(find mobile_robot_description)/urdf/ackermann_steering.xacro" /> -->
 <xacro:include filename="$(find mobile_robot_description)/urdf/gazebo.xacro" />
@@ -28,7 +28,8 @@
 </joint> -->
 <joint name="lidar1_joint" type="fixed">
-    <parent link="Lidar1"/>
+    <parent link="chassis"/>
     <child link="Lidar1_link"/>
-    <origin xyz="0.015 0.0 0.06" rpy="0.0 0.0 0.0"/>
+    <origin xyz="0.0 0.0 0.1" rpy="0.0 0.0 0.0"/>
+    <!-- <origin xyz="0.3402 0.0261 -0.0248" rpy="0.0 0.0 0.0"/> -->
 </joint>
 <!-- <joint name="lidar2_joint" type="fixed">

Commit message: Update lidar1_joint position in mobile_robot.urdf.xacro to adjust height

File: mobile_robot_description/urdf/mobile_robot.urdf.xacro (robot description, xacro)
@@ -30,5 +30,5 @@
     <parent link="chassis"/>
     <child link="Lidar1_link"/>
-    <origin xyz="0.0 0.0 0.1" rpy="0.0 0.0 0.0"/>
+    <origin xyz="0.0 0.0 0.3" rpy="0.0 0.0 0.0"/>
     <!-- <origin xyz="0.3402 0.0261 -0.0248" rpy="0.0 0.0 0.0"/> -->
 </joint>

Commit message: Remove unused URDF and SDF files for diff drive, ackermann steering, camera, and empty world

File: mobile_robot_description/urdf/mobile_robot.urdf.xacro (robot description, xacro)
@@ -4,8 +4,5 @@
 <xacro:include filename="$(find mobile_robot_description)/urdf/materials.xacro" />
 <xacro:include filename="$(find mobile_robot_description)/urdf/mobile_robot.xacro" />
-<!-- <xacro:include filename="$(find mobile_robot_description)/urdf/camera.xacro" /> -->
 <xacro:include filename="$(find mobile_robot_description)/urdf/lidar.xacro" />
-<!-- <xacro:include filename="$(find mobile_robot_description)/urdf/diff_drive.xacro" /> -->
-<!-- <xacro:include filename="$(find mobile_robot_description)/urdf/ackermann_steering.xacro" /> -->
 <xacro:include filename="$(find mobile_robot_description)/urdf/gazebo.xacro" />
 <xacro:include filename="$(find mobile_robot_description)/urdf/mobile_robot.ros2_control.xacro" />
@@ -22,19 +19,8 @@
     <origin xyz="0.0 0.0 0.0" rpy="0.0 0.0 0.0"/>
 </joint>
-<!-- <joint name="camera_joint" type="fixed">
-    <parent link="IntelRealsense_D435_Multibody"/>
-    <child link="Camera"/>
-    <origin xyz="0.01 0.0 0.00" rpy="0.0 0.0 0.0"/>
-</joint> -->
 <joint name="lidar1_joint" type="fixed">
     <parent link="chassis"/>
     <child link="Lidar1_link"/>
     <origin xyz="0.0 0.0 0.3" rpy="0.0 0.0 0.0"/>
-    <!-- <origin xyz="0.3402 0.0261 -0.0248" rpy="0.0 0.0 0.0"/> -->
 </joint>
-<!-- <joint name="lidar2_joint" type="fixed">
-    <parent link="Lidar2"/>
-    <child link="Lidar2_link"/>
-    <origin xyz="-0.015 0.0 0.06" rpy="0.0 0.0 0.0"/>
-</joint> -->
 </robot>
